File: ReadTemperature/ReadTemperature.brd (EAGLE design)
At the start: 140.3 x 59.7 mm, 2 parts, among them U1 ARDUINO-UNO-R3-SHIELD, U2 TMP36GT9Z_TO92

Commit message: Update temperature reading program
Connections:
- removed net U1_D2: U1.D2, U2.2
- new net U1_D7: U1.D7, U2.3
- net U1_5V: now also U2.2; no longer U2.3
Changed lines of the file:
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@@
 <wire x1="134.2272" y1="24.1106" x2="52.965" y2="5.715" width="0" layer="19" extent="1-1"/>
 </signal>
-<signal name="U1_D2">
+<signal name="U1_5V">
 <contactref element="U2" pad="2"/>
-<contactref element="U1" pad="D2"/>
-<wire x1="136.1322" y1="22.8406" x2="68.205" y2="53.975" width="0" layer="19" extent="1-1"/>
+<contactref element="U1" pad="5V"/>
+<wire x1="136.1322" y1="22.8406" x2="47.885" y2="5.715" width="0" layer="19" extent="1-1"/>
 </signal>
-<signal name="U1_5V">
+<signal name="U1_D7">
 <contactref element="U2" pad="3"/>
-<contactref element="U1" pad="5V"/>
-<wire x1="134.2272" y1="21.5706" x2="47.885" y2="5.715" width="0" layer="19" extent="1-1"/>
+<contactref element="U1" pad="D7"/>
+<wire x1="134.2272" y1="21.5706" x2="55.505" y2="53.975" width="0" layer="19" extent="1-1"/>
 </signal>
 </signals>
